Commit message: URDF viewable, orientation bugs

File: ros_ws/src/robot_description/urdf/robot.urdf (robot description, URDF)
Before this commit: robot robot_config, 3 links, 2 joints
Links:
- link body: geometry collision mesh filename=package://robot_description/assets/body.stl; visual mesh filename=package://robot_description/assets/body.stl
- link left_wheel: geometry collision mesh filename=package://robot_description/assets/left_wheel.stl; visual mesh filename=package://robot_description/assets/left_wheel.stl
- link right_wheel: geometry collision mesh filename=package://robot_description/assets/right_wheel.stl; visual mesh filename=package://robot_description/assets/right_wheel.stl

Commit message: Fully Drivable

File: ros_ws/src/robot_description/urdf/robot.urdf (robot description, URDF)
Before this commit: robot robot_config, 3 links, 2 joints
Links:
- added link base_link
Joints:
- added joint base_to_body: type fixed, parent base_link, child body, origin xyz=0 0 0 rpy=0 0 -1.5708

Commit message: simulate with gazebo

File: ros_ws/src/robot_description/urdf/robot.urdf (robot description, URDF)
Before this commit: robot robot_config, 4 links, 3 joints
Joints:
- joint base_to_body: origin xyz=0 0 0 rpy=0 0 -1.5708 -> xyz=0 0 0 rpy=0 0 0
